File: SD2SP2-Pro 2.0/Kicad/Outer/Gamecube_SD2SP2PRO.kicad_sch (KiCad schematic)
At the start: 4 parts, among them J2 Conn_02x04_Odd_Even, J3 Micro_SD_Card, U1 74AHC1G32

Commit message: updated schematic
Parts:
- C1: value 100n -> 22u
Changed lines of the file:
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@@
 			)
 		)
-		(property "Value" "100n"
+		(property "Value" "22u"
 			(at 164.8968 106.299 0)
 			(effects

Commit message: added LCSC alt part#
Parts:
- U1: LCSC Part (none) -> C12488
Changed lines of the file:
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@@
 			)
 		)
-		(property "Datasheet" "http://www.ti.com/lit/sg/scyt129e/scyt129e.pdf"
+		(property "Datasheet" ""
 			(at 96.52 109.22 0)
 			(effects
@@
 			(effects
 				(font
+					(size 1.27 1.27)
+				)
+				(hide yes)
+			)
+		)
+		(property "LCSC Part" "C12488"
+			(at 96.52 109.22 90)
+			(effects
+				(font
